File: speedster-crossover.sch (KiCad schematic (older format))
At the start: 10 parts, among them X1 HIGH-PASS IN, X2 LOW-PASS IN

Commit message: add schematic image
Parts:
- X1: value HIGH-PASS IN -> HIGH-PASS
- X2: value LOW-PASS IN -> LOW-PASS
Changed lines of the file:
@@
 P 7300 3900
 F 0 "X1" H 7300 4150 50  0000 C CNN
-F 1 "HIGH-PASS IN" V 7400 3900 50  0000 C CNN
+F 1 "HIGH-PASS" V 7400 3900 50  0000 C CNN
 F 2 "components:OAL_pheonix_mkds_2.5-4pos" H 7300 3900 50  0001 C CNN
 F 3 "" H 7300 3900 50  0000 C CNN
@@
 P 7300 4550
 F 0 "X2" H 7300 4900 50  0000 C CNN
-F 1 "LOW-PASS IN" V 7400 4550 50  0000 C CNN
+F 1 "LOW-PASS" V 7400 4550 50  0000 C CNN
 F 2 "components:OAL_pheonix_mkds_2.5-6pos" H 7300 4550 50  0001 C CNN
 F 3 "" H 7300 4550 50  0000 C CNN
